Commit message: updated jetbot_description with camera and LiDAR; separated gazebo plugins from URDF; added a launch file just for the description so that can be used and loaded in other launch files

File: jetbot_description/urdf/jetbot.urdf (robot description, URDF)
Before this commit: robot JetBot, 4 links, 3 joints
Links:
- removed link JetBot__camera_link
- removed link JetBot__chassis
- removed link JetBot__left_wheel
- removed link JetBot__right_wheel
- added link base_footprint
- added link base_link, mass 1.0; collision mesh filename=package://jetbot_description/meshes/JetBot-v3-Chassis.dae scale=0.001 0.001 0.001; visual mesh filename=package://jetbot_description/meshes/JetBot-v3-Chassis.dae scale=0.001 0.001 0.001
- added link camera_link, mass 0.01; visual box size=0.001 0.001 0.001
- added link left_wheel, mass 0.1; collision cylinder length=0.008 radius=0.030; visual mesh filename=package://jetbot_description/meshes/JetBot-v3-Wheel.stl scale=0.001 0.001 0.001
- added link lidar_link, mass 0.0; collision mesh filename=package://jetbot_description/meshes/lidar-base.dae scale=1.0 1.0 1.0; visual mesh filename=package://jetbot_description/meshes/lidar-base.dae scale=1.0 1.0 1.0
- added link right_wheel, mass 0.1; collision cylinder length=0.008 radius=0.030; visual mesh filename=package://jetbot_description/meshes/JetBot-v3-Wheel.stl scale=0.001 0.001 0.001
Joints:
- removed joint JetBot__camera_joint
- removed joint JetBot__left_wheel_hinge
- removed joint JetBot__right_wheel_hinge
- added joint base_joint: type fixed, parent base_footprint, child base_link, origin xyz=0.0 0.0 0.010 rpy=0 0 0
- added joint camera_joint: type fixed, parent base_link, child camera_link, origin xyz=0.065   0      0.0857 rpy=0    0.25  0, axis 0.96891  0       0.2474
- added joint left_wheel_hinge: type continuous, parent base_link, child left_wheel, origin xyz=0.03     0.05125  0.03 rpy=0       0       1.57079, axis 1  0  0
- added joint lidar_joint: type fixed, parent base_link, child lidar_link, origin xyz=0.0 -0.0058  0.127 rpy=0   0   3.14, axis 0 0 0
- added joint right_wheel_hinge: type continuous, parent base_link, child right_wheel, origin xyz=0.03   -0.0595  0.03 rpy=0       0       1.57079, axis 1  0  0
